File: uECG_v4_5/uECG_v4_5.kicad_pcb (KiCad board)
At the start: 2 copper layers, 63 x 22 mm, 72 parts, among them IC1 BMI160, IC2 AD8606ARMZ, IC3 SIP32510DT-T1-GE3, IC4 SIP32510DT-T1-GE3, J2 USB_B_Micro, J5 Conn_01x01_Male, J6 Conn_01x01_Male, SW1 SW_Push, SW2 SW_SPDT, U1 nRF52832-QFxx, U2 MCP3911(QFN), U3 74AHC1G32, U4 MCP73831-2-OT, U5 XC6206P332MR_SOT23, U6 XC6206P302MR_SOT23, Y1 32MHz

Commit message: ADD: kicad version 6
Other:
- net class Default removed
